Commit message: wip

File: src/turtlebot3/turtlebot3_description/urdf/turtlebot3_burger.urdf.xacro (robot description, xacro)
@@ -43,5 +43,5 @@
         <mesh filename="package://turtlebot3_description/meshes/wheels/left_tire.dae" scale="0.001 0.001 0.001"/>
       </geometry>
-      <material name="dark"/>
+      <material name="red"/>
     </visual>
     <collision>
@@ -71,5 +71,5 @@
         <mesh filename="package://turtlebot3_description/meshes/wheels/right_tire.dae" scale="0.001 0.001 0.001"/>
       </geometry>
-      <material name="dark"/>
+      <material name="red"/>
     </visual>
     <collision>
@@ -124,5 +124,5 @@
         <mesh filename="package://turtlebot3_description/meshes/sensors/lds.dae" scale="0.001 0.001 0.001"/>
       </geometry>
-      <material name="dark"/>
+      <material name="red"/>
     </visual>
     <collision>
